Commit message: improved parameters
Signed-off-by: Yuri van Warmerdam <yuri.van.warmerdam@alliander.com>

File: rcdt_utilities/urdf/rcdt_realsense_d435.urdf.xacro (robot description, xacro)
@@ -4,8 +4,9 @@
 SPDX-License-Identifier: Apache-2.0
 -->
-<robot xmlns:xacro="http://www.ros.org/wiki/xacro" name="p">
-  <xacro:macro name="p">
-    <xacro:property name="parent" default="world" />
-    <xacro:property name="simulation" default="false" />
+<robot xmlns:xacro="http://www.ros.org/wiki/xacro" name="realsense_d435">
+  <xacro:macro name="realsense_d435">
+    <xacro:arg name="simulation" default="false" />
+    <xacro:arg name="parent" default="world" />
+    <xacro:property name="parent" value="$(arg parent)"/>
     <xacro:include filename="$(find realsense2_description)/urdf/_d435.urdf.xacro" />
     <xacro:sensor_d435
@@ -16,8 +17,8 @@
     <xacro:if value="${parent != ''}">
       <xacro:if value="${parent == 'world'}">
-        <link name="${parent}" />
+        <link name="$(arg parent)" />
       </xacro:if>
     </xacro:if>
-    <!-- <xacro:if value="${simulation}"> -->
+    <xacro:if value="$(arg simulation)">
     <gazebo reference="camera_color_frame">
       <sensor type="camera" name="intel_realsense_d435_color">
@@ -63,6 +64,6 @@
       </sensor>
     </gazebo>
-    <!-- </xacro:if> -->
+    </xacro:if>
   </xacro:macro>
-  <xacro:p></xacro:p>
+  <xacro:realsense_d435></xacro:realsense_d435>
 </robot>

Commit message: Fix topic names and depth camera.
Signed-off-by: Jelmer de Wolde <jelmer.de.wolde@alliander.com>

File: rcdt_utilities/urdf/rcdt_realsense_d435.urdf.xacro (robot description, xacro)
@@ -5,63 +5,74 @@
 -->
 <robot xmlns:xacro="http://www.ros.org/wiki/xacro" name="realsense_d435">
-  <xacro:macro name="realsense_d435">
-    <xacro:arg name="simulation" default="false" />
-    <xacro:arg name="parent" default="world" />
-    <xacro:property name="parent" value="$(arg parent)"/>
+  <xacro:macro name="realsense_d435"
+    params="
+    simulation:=true
+    parent:=world
+    namespace:=camera
+    ">
+    <!-- Create world link if this is the parent: -->
+    <xacro:if value="${parent == 'world'}">
+      <link name="${parent}" />
+    </xacro:if>
+    <!-- Create camera link and connect to parent: -->
+    <link name="test" />
+    <joint name="test_joint" type="fixed">
+      <parent link="${parent}" />
+      <child link="test" />
+    </joint>
+    <!-- Include realsense xacro: -->
     <xacro:include filename="$(find realsense2_description)/urdf/_d435.urdf.xacro" />
     <xacro:sensor_d435
-      parent="${parent}"
+      parent="test"
       use_nominal_extrinsics="true">
       <origin xyz="0 0 0" rpy="0 0 0" />
     </xacro:sensor_d435>
-    <xacro:if value="${parent != ''}">
-      <xacro:if value="${parent == 'world'}">
-        <link name="$(arg parent)" />
-      </xacro:if>
-    </xacro:if>
-    <xacro:if value="$(arg simulation)">
-    <gazebo reference="camera_color_frame">
-      <sensor type="camera" name="intel_realsense_d435_color">
-        <always_on>true</always_on>
-        <update_rate>30.0</update_rate>
-        <topic>some_name/color/image_raw</topic>
-        <visualize>false</visualize>
-        <ignition_frame_id>name_color_optical_frame</ignition_frame_id>
-        <horizontal_fov>${69.0/180.0*pi}</horizontal_fov>
-        <image>
-          <width>1280</width>
-          <height>720</height>
-          <format>R8G8B8</format>
-        </image>
-        <clip>
-          <near>0.02</near>
-          <far>300.0</far>
-        </clip>
-      </sensor>
-      <sensor type="depth_camera" name="ns_namespace_intel_realsense_d435_depth">
-        <always_on>true</always_on>
-        <update_rate>30.0</update_rate>
-        <topic>ns/namespace/depth/image_rect_raw</topic>
-        <visualize>false</visualize>
-        <ignition_frame_id>namespace_depth_optical_frame</ignition_frame_id>
-        <camera>
-          <horizontal_fov>${87.0/180.0*pi}</horizontal_fov>
+    <!-- Add gazebo plugin: -->
+    <xacro:if value="${simulation}">
+      <gazebo reference="${namespace}_link">
+        <!-- rgb_camera: -->
+        <sensor type="camera" name="${namespace}_intel_realsense_d435_color">
+          <always_on>true</always_on>
+          <update_rate>30.0</update_rate>
+          <topic>${namespace}/color/image_raw</topic>
+          <visualize>false</visualize>
+          <ignition_frame_id>${namespace}_color_optical_frame</ignition_frame_id>
+          <horizontal_fov>${69.0/180.0*pi}</horizontal_fov>
           <image>
             <width>1280</width>
             <height>720</height>
-            <format>R_FLOAT32</format>
+            <format>R8G8B8</format>
           </image>
           <clip>
-            <near>0.28</near>
-            <far>8.0</far>
+            <near>0.02</near>
+            <far>300.0</far>
           </clip>
-          <noise>
-            <type>gaussian</type>
-            <mean>0.0</mean>
-            <stddev>0.005</stddev>
-          </noise>
-        </camera>
-      </sensor>
-    </gazebo>
+        </sensor>
+        <!-- depth camera -->
+        <sensor type="depth_camera" name="${namespace}_intel_realsense_d435_depth">
+          <always_on>true</always_on>
+          <update_rate>30.0</update_rate>
+          <topic>${namespace}/depth/image_rect_raw</topic>
+          <visualize>false</visualize>
+          <ignition_frame_id>${namespace}_depth_optical_frame</ignition_frame_id>
+          <camera>
+            <horizontal_fov>${87.0/180.0*pi}</horizontal_fov>
+            <image>
+              <width>1280</width>
+              <height>720</height>
+              <format>R_FLOAT32</format>
+            </image>
+            <clip>
+              <near>0.28</near>
+              <far>8.0</far>
+            </clip>
+            <noise>
+              <type>gaussian</type>
+              <mean>0.0</mean>
+              <stddev>0.005</stddev>
+            </noise>
+          </camera>
+        </sensor>
+      </gazebo>
     </xacro:if>
   </xacro:macro>

Commit message: Fix for use with franka.
Signed-off-by: Jelmer de Wolde <jelmer.de.wolde@alliander.com>

File: rcdt_utilities/urdf/rcdt_realsense_d435.urdf.xacro (robot description, xacro)
@@ -4,8 +4,8 @@
 SPDX-License-Identifier: Apache-2.0
 -->
-<robot xmlns:xacro="http://www.ros.org/wiki/xacro" name="realsense_d435">
-  <xacro:macro name="realsense_d435"
+<robot xmlns:xacro="http://www.ros.org/wiki/xacro" name="rcdt_realsense_d435">
+  <xacro:macro name="rcdt_realsense_d435"
     params="
-    simulation:=true
+    gazebo:=true
     parent:=world
     namespace:=camera
@@ -15,19 +15,13 @@
       <link name="${parent}" />
     </xacro:if>
-    <!-- Create camera link and connect to parent: -->
-    <link name="test" />
-    <joint name="test_joint" type="fixed">
-      <parent link="${parent}" />
-      <child link="test" />
-    </joint>
     <!-- Include realsense xacro: -->
     <xacro:include filename="$(find realsense2_description)/urdf/_d435.urdf.xacro" />
     <xacro:sensor_d435
-      parent="test"
+      parent="${parent}"
       use_nominal_extrinsics="true">
       <origin xyz="0 0 0" rpy="0 0 0" />
     </xacro:sensor_d435>
     <!-- Add gazebo plugin: -->
-    <xacro:if value="${simulation}">
+    <xacro:if value="${gazebo}">
       <gazebo reference="${namespace}_link">
         <!-- rgb_camera: -->
@@ -55,5 +49,5 @@
           <topic>${namespace}/depth/image_rect_raw</topic>
           <visualize>false</visualize>
-          <ignition_frame_id>${namespace}_depth_optical_frame</ignition_frame_id>
+          <ignition_frame_id>${namespace}_depth_frame</ignition_frame_id>
           <camera>
             <horizontal_fov>${87.0/180.0*pi}</horizontal_fov>
@@ -77,4 +71,3 @@
     </xacro:if>
   </xacro:macro>
-  <xacro:realsense_d435></xacro:realsense_d435>
 </robot>
